File: binary_clock_PCB/binary_clock.kicad_pcb (KiCad board)
At the start: 2 copper layers, 9 parts, among them U1 ESP32-S3R8, U2 AP2112K-3.3, U2 W25Q128JVPIQ, U3 MAX-M10S, U4 ESP32-WROOM-32E-R2, U5 SN74LVC1T45GW

Commit message: Update
Parts:
- removed the U2 at (101.2, 90.6)
- added U6: DS3231M, Package_SO:SOIC-16W_7.5x10.3mm_P1.27mm, F.Cu at (33.5, 100.2)
- U1: value ESP32-S3R8 -> ESP32-S3-WROOM-2-N32R8V; footprint Package_DFN_QFN:QFN-56-1EP_7x7mm_P0.4mm_EP4x4mm -> RF_Module:ESP32-S3-WROOM-2
- U4: value ESP32-WROOM-32E-R2 -> PCF8523TK; footprint RF_Module:ESP32-WROOM-32D -> Package_SON:HVSON-8-1EP_4x4mm_P0.8mm_EP2.2x3.1mm
- U5: footprint Package_TO_SOT_SMD:SOT-563 -> Package_TO_SOT_SMD:SOT-363_SC-70-6
- moved U4 97.6 mm to (27.4, 110.5)
- moved U1 28.0 mm to (109.1, 65.0)
Connections:
- U1 pad 1: unconnected-(U1-LNA_IN-Pad1) -> GND
- U1 pad 13: unconnected-(U1-GPIO8-Pad13) -> /D-
- U1 pad 14: unconnected-(U1-GPIO9-Pad14) -> /D+
- U1 pad 2: Net-(U1-VDD3P3-Pad2) -> 3V3
- U1 pad 3: Net-(U1-VDD3P3-Pad2) -> unconnected-(U1-EN-Pad3)
- U1 pad 40: unconnected-(U1-GPIO35-Pad40) -> GND
- U1 pad 41: unconnected-(U1-GPIO36-Pad41) -> GND
- U4 pad 1: Net-(U4-GND-Pad1) -> unconnected-(U4-OSCI-Pad1)
- U4 pad 4: unconnected-(U4-SENSOR_VP-Pad4) -> Net-(U4-VSS-Pad4)
- U4 pad 9: unconnected-(U4-IO33-Pad9) -> Net-(U4-VSS-Pad4)
- U5 pad 1: unconnected-(U5-VCCA-Pad1) -> 3V3
- U5 pad 2: unconnected-(U5-GND-Pad2) -> GND
- U5 pad 5: unconnected-(U5-DIR-Pad5) -> /VBUS
- U5 pad 6: unconnected-(U5-VCCB-Pad6) -> /VBUS

Commit message: Update
Parts:
- removed the D2 at (54.6, 57.9)
- removed U4: PCF8523TK, Package_SON:HVSON-8-1EP_4x4mm_P0.8mm_EP2.2x3.1mm
- added D4: SK6812, LED_SMD:LED_SK6812_PLCC4_5.0x5.0mm_P3.2mm, F.Cu at (155.3, 64.4)
- added U7: AP2112K-3.3, Package_TO_SOT_SMD:SOT-23-5, F.Cu at (59.4, 109.0)
- moved U1 20.9 mm to (118.1, 46.2)
Connections:
- U1 pad 15: unconnected-(U1-IO3-Pad15) -> /SDA
- U1 pad 17: unconnected-(U1-IO9-Pad17) -> /NEO_MCU
- U1 pad 2: 3V3 -> 3V3_MCU
- U1 pad 27: unconnected-(U1-IO0-Pad27) -> /BOOT
- U1 pad 3: unconnected-(U1-EN-Pad3) -> /RESET
- U1 pad 38: unconnected-(U1-IO2-Pad38) -> /SCL
- U1 pad 4: unconnected-(U1-IO4-Pad4) -> /NEO
- U1 pad 5: unconnected-(U1-IO5-Pad5) -> /PPS
- U1 pad 7: unconnected-(U1-IO7-Pad7) -> /3V_EN
- U2 pad 5: 3V3 -> 3V3_MCU
- U3 pad 1: Net-(U3-GND-Pad1) -> GND
- U3 pad 10: Net-(U3-GND-Pad1) -> GND
- U3 pad 11: unconnected-(U3-RF_IN-Pad11) -> Net-(J2-In)
- U3 pad 12: Net-(U3-GND-Pad1) -> GND
- U3 pad 16: unconnected-(U3-SDA-Pad16) -> /SDA
- U3 pad 17: unconnected-(U3-SCL-Pad17) -> /SCL
- U3 pad 4: unconnected-(U3-TIMEPULSE-Pad4) -> /PPS
- U3 pad 7: unconnected-(U3-VCC_IO-Pad7) -> 3V3
- U3 pad 8: unconnected-(U3-VCC-Pad8) -> 3V3
- U5 pad 3: unconnected-(U5-A-Pad3) -> /NEO
- U5 pad 4: unconnected-(U5-B-Pad4) -> /NEO_5V
- U6 pad 10: Net-(U6-GND-Pad10) -> GND
- U6 pad 11: Net-(U6-GND-Pad10) -> GND
- U6 pad 12: Net-(U6-GND-Pad10) -> GND
- U6 pad 13: Net-(U6-GND-Pad10) -> GND
- U6 pad 14: unconnected-(U6-VBAT-Pad14) -> GND
- U6 pad 15: unconnected-(U6-SDA-Pad15) -> /SDA
- U6 pad 16: unconnected-(U6-SCL-Pad16) -> /SCL
- U6 pad 2: unconnected-(U6-VCC-Pad2) -> Net-(U6-VCC)
- U6 pad 5: Net-(U6-GND-Pad10) -> GND
- U6 pad 6: Net-(U6-GND-Pad10) -> GND
- U6 pad 7: Net-(U6-GND-Pad10) -> GND
- U6 pad 8: Net-(U6-GND-Pad10) -> GND
- U6 pad 9: Net-(U6-GND-Pad10) -> GND

Commit message: Update gitignore, PCB
Parts:
- added C1: 1uF, Capacitor_SMD:C_0603_1608Metric, F.Cu at (64.5, 141.7)
- added C10: 100nF, Capacitor_SMD:C_0603_1608Metric, F.Cu at (64.2, 128.0)
- added C11: 100nF, Capacitor_SMD:C_0603_1608Metric, F.Cu at (64.5, 134.1)
- added C12: 100nF, Capacitor_SMD:C_0603_1608Metric, F.Cu at (64.5, 139.1)
- added C13: 100nF, Capacitor_SMD:C_0603_1608Metric, F.Cu at (64.5, 146.7)
- added C14: 100nF, Capacitor_SMD:C_0603_1608Metric, F.Cu at (68.5, 131.6)
- added C15: 100nF, Capacitor_SMD:C_0603_1608Metric, F.Cu at (68.5, 134.1)
- added C16: 100nF, Capacitor_SMD:C_0603_1608Metric, F.Cu at (68.5, 136.6)
- added C17: 100nF, Capacitor_SMD:C_0603_1608Metric, F.Cu at (68.5, 139.1)
- added C18: 100nF, Capacitor_SMD:C_0603_1608Metric, F.Cu at (68.5, 144.2)
- added C19: 100nF, Capacitor_SMD:C_0603_1608Metric, F.Cu at (68.5, 146.7)
- added C2: 10uF, Capacitor_SMD:C_0603_1608Metric, F.Cu at (64.5, 136.6)
- added C20: 100nF, Capacitor_SMD:C_0603_1608Metric, F.Cu at (72.5, 139.1)
- added C21: 100nF, Capacitor_SMD:C_0603_1608Metric, F.Cu at (72.5, 141.7)
- added C22: 100nF, Capacitor_SMD:C_0603_1608Metric, F.Cu at (72.5, 146.7)
- added C23: 100nF, Capacitor_SMD:C_0603_1608Metric, F.Cu at (76.5, 134.1)
- added C24: 100nF, Capacitor_SMD:C_0603_1608Metric, F.Cu at (76.5, 136.6)
- added C25: 100nF, Capacitor_SMD:C_0603_1608Metric, F.Cu at (76.5, 139.1)
- added C26: 100nF, Capacitor_SMD:C_0603_1608Metric, F.Cu at (76.5, 141.7)
- added C27: 100nF, Capacitor_SMD:C_0603_1608Metric, F.Cu at (76.5, 144.2)
- added C3: 10uF, Capacitor_SMD:C_0603_1608Metric, F.Cu at (64.5, 144.2)
- added C4: 10uF, Capacitor_SMD:C_0603_1608Metric, F.Cu at (68.5, 141.7)
- added C5: 10uF, Capacitor_SMD:C_0603_1608Metric, F.Cu at (72.5, 134.1)
- added C6: 100nF, Capacitor_SMD:C_0603_1608Metric, F.Cu at (72.5, 131.6)
- added C7: 100nF, Capacitor_SMD:C_0603_1608Metric, F.Cu at (76.5, 131.6)
- added C8: 1uF, Capacitor_SMD:C_0603_1608Metric, F.Cu at (72.5, 136.6)
- added C9: 1uF, Capacitor_SMD:C_0603_1608Metric, F.Cu at (72.5, 144.2)
- added D10: SK6812, LED_SMD:LED_SK6812_PLCC4_5.0x5.0mm_P3.2mm, F.Cu at (49.9, 133.7)
- added D11: SK6812, LED_SMD:LED_SK6812_PLCC4_5.0x5.0mm_P3.2mm, F.Cu at (49.9, 140.3)
- added D12: SK6812, LED_SMD:LED_SK6812_PLCC4_5.0x5.0mm_P3.2mm, F.Cu at (49.9, 146.9)
- added D13: SK6812, LED_SMD:LED_SK6812_PLCC4_5.0x5.0mm_P3.2mm, F.Cu at (49.9, 153.5)
- added D14: SK6812, LED_SMD:LED_SK6812_PLCC4_5.0x5.0mm_P3.2mm, F.Cu at (49.9, 160.2)
- added D15: SK6812, LED_SMD:LED_SK6812_PLCC4_5.0x5.0mm_P3.2mm, F.Cu at (49.9, 166.8)
- added D16: SK6812, LED_SMD:LED_SK6812_PLCC4_5.0x5.0mm_P3.2mm, F.Cu at (58.3, 133.7)
- added D17: SK6812, LED_SMD:LED_SK6812_PLCC4_5.0x5.0mm_P3.2mm, F.Cu at (58.3, 140.3)
- added D18: SK6812, LED_SMD:LED_SK6812_PLCC4_5.0x5.0mm_P3.2mm, F.Cu at (58.3, 146.9)
- added D19: SK6812, LED_SMD:LED_SK6812_PLCC4_5.0x5.0mm_P3.2mm, F.Cu at (58.3, 153.5)
- added D20: SK6812, LED_SMD:LED_SK6812_PLCC4_5.0x5.0mm_P3.2mm, F.Cu at (58.3, 160.2)
- added D4: SK6812, LED_SMD:LED_SK6812_PLCC4_5.0x5.0mm_P3.2mm, F.Cu at (41.5, 133.7)
- added D5: SK6812, LED_SMD:LED_SK6812_PLCC4_5.0x5.0mm_P3.2mm, F.Cu at (41.5, 140.3)
- added D6: SK6812, LED_SMD:LED_SK6812_PLCC4_5.0x5.0mm_P3.2mm, F.Cu at (41.5, 146.9)
- added D7: SK6812, LED_SMD:LED_SK6812_PLCC4_5.0x5.0mm_P3.2mm, F.Cu at (41.5, 153.5)
- added D8: SK6812, LED_SMD:LED_SK6812_PLCC4_5.0x5.0mm_P3.2mm, F.Cu at (41.5, 160.2)
- added D9: SK6812, LED_SMD:LED_SK6812_PLCC4_5.0x5.0mm_P3.2mm, F.Cu at (41.5, 166.8)
- added J3: Conn_01x08_Socket, Connector_PinHeader_2.54mm:PinHeader_1x08_P2.54mm_Vertical, F.Cu at (61.3, 65.7)
- added JP1: SolderJumper_2_Bridged, besser_footprints:solder_jumper_bridged, F.Cu at (68.2, 56.5)
- added JP2: SolderJumper_2_Bridged, besser_footprints:solder_jumper_bridged, F.Cu at (68.2, 59.8)
- added JP3: SolderJumper_2_Bridged, besser_footprints:solder_jumper_bridged, F.Cu at (101.4, 132.0)
- added R1: 5.1K, Capacitor_SMD:C_0603_1608Metric, F.Cu at (73.7, 80.7)
- added R2: 5.1K, Capacitor_SMD:C_0603_1608Metric, F.Cu at (73.7, 83.2)
- added R3: 5.1K, Capacitor_SMD:C_0603_1608Metric, F.Cu at (73.7, 88.2)
- added R4: 5.1K, Capacitor_SMD:C_0603_1608Metric, F.Cu at (73.7, 85.7)
- added R5: 5.1K, Capacitor_SMD:C_0603_1608Metric, F.Cu at (73.7, 90.8)
- renumbered D4 to D1, D1 to D3, U7 to U3, U3 to U4, U6 to U5, U5 to U7
Connections:
- net /NEO renamed /NEO_DISP
- net /VBUS renamed VBUS
- D3 pad 1: unconnected-(D1-VSS-Pad1) -> GND
- D3 pad 2: unconnected-(D1-DIN-Pad2) -> /NEO_5VLL
- D3 pad 3: unconnected-(D1-VDD-Pad3) -> Net-(D10-VDD)
- D3 pad 4: unconnected-(D1-DOUT-Pad4) (its old number) -> Net-(D3-DOUT)
- U1 pad 17: /NEO_MCU -> unconnected-(U1-IO9-Pad17)
- U1 pad 18: unconnected-(U1-IO10-Pad18) -> /IO10
- U1 pad 19: unconnected-(U1-IO11-Pad19) -> /IO11
- U1 pad 20: unconnected-(U1-IO12-Pad20) -> /IO12
- U1 pad 21: unconnected-(U1-IO13-Pad21) -> /IO13
- U1 pad 22: unconnected-(U1-IO14-Pad22) -> /IO14
- U1 pad 36: unconnected-(U1-RXD0/IO44-Pad36) -> /M_RX
- U1 pad 37: unconnected-(U1-TXD0/IO43-Pad37) -> /M_TX
- U1 pad 6: unconnected-(U1-IO6-Pad6) -> /NEO_MCU
- U4 pad 2: unconnected-(U3-TXD-Pad2) -> Net-(JP2-B)
- U4 pad 3: unconnected-(U3-RXD-Pad3) -> Net-(JP1-B)
- U5 pad 2: Net-(U6-VCC) -> 3V3
- U7 pad 4: /NEO_5V -> /NEO_5VLL

Commit message: Update PCB
Parts:
- added C9: 1uF, Capacitor_SMD:C_0603_1608Metric, F.Cu at (69.8, 41.2)
- added J1: USB4105-GF-A, Connector_USB:USB_C_Receptacle_GCT_USB4105-xx-A_16P_TopMnt_Horizontal, F.Cu at (40.8, 72.0)
- added J2: uFL, Connector_Coaxial:U.FL_Hirose_U.FL-R-SMT-1_Vertical, F.Cu at (38.8, 86.3)
- added J4: JST-SM04B-SRSS, besser_footprints:JST_SH_SM04B-SRSS-TB_1x04-1MP_P1.00mm_Horizontal, F.Cu at (72.0, 32.6)
- added J5: JST-SM04B-SRSS, besser_footprints:JST_SH_SM04B-SRSS-TB_1x04-1MP_P1.00mm_Horizontal, F.Cu at (69.8, 19.2)
- added J6: JST-SM04B-SRSS, besser_footprints:JST_SH_SM04B-SRSS-TB_1x04-1MP_P1.00mm_Horizontal, F.Cu at (42.2, 23.4)
- added U6: VEML7700-TT, besser_footprints:VEML7700, F.Cu at (26.5, 46.3)
- added U8: VEML7700-TT, besser_footprints:VEML7700, F.Cu at (21.7, 64.8)
Connections:
- C9 pad 1: GND -> 3V3
- C9 pad 2: 3V3 -> GND
Other:
- board text added: "2²"

Commit message: Start on PCB
Parts:
- removed the C9 at (72.5, 144.2)
- removed the C9 at (69.8, 41.2)
- added C9: 1uF, Capacitor_SMD:C_0603_1608Metric, F.Cu at (53.2, 182.6)
- added SW1: PTS636 SK25F, Button_Switch_SMD:SW_Tactile_SPST_NO_Straight_CK_PTS636Sx25SMTRLFS, F.Cu at (56.5, 186.5)
- added SW2: PTS636 SK25F, Button_Switch_SMD:SW_Tactile_SPST_NO_Straight_CK_PTS636Sx25SMTRLFS, F.Cu at (56.5, 191.8)
- J1, U1: moved to B.Cu
- moved J1 235.3 mm to (275.0, 50.0), turned to -90 degrees
- moved J6 159.7 mm to (71.7, 180.3)
- moved J5 153.5 mm to (71.7, 172.7)
- moved U6 149.1 mm to (72.0, 188.2)
- moved D3 142.9 mm to (47.0, 190.4), turned to 180 degrees
- moved U8 138.0 mm to (72.0, 193.3)
- moved J4 132.5 mm to (71.7, 165.1)
- moved JP1 129.1 mm to (63.7, 185.5)
- moved JP2 129.1 mm to (63.7, 188.7)
- moved U7 110.6 mm to (74.5, 154.4)
- moved J3 99.4 mm to (78.4, 163.6)
- moved U2 93.6 mm to (78.1, 186.5)
- moved D1 93.5 mm to (62.0, 58.0)
- moved R4 84.8 mm to (65.2, 170.1)
- moved U3 84.2 mm to (78.1, 191.2)
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Connections:
- net Net-(J1-CC1) renamed /CC1
- net Net-(J1-CC2) renamed /CC2
- net Net-(J2-In) renamed /ANT
- D10 pad 3: Net-(D10-VDD) -> VBUS
- D11 pad 3: Net-(D10-VDD) -> VBUS
- D12 pad 3: Net-(D10-VDD) -> VBUS
- D13 pad 3: Net-(D10-VDD) -> VBUS
- D14 pad 3: Net-(D10-VDD) -> VBUS
- D15 pad 3: Net-(D10-VDD) -> VBUS
- D16 pad 3: Net-(D10-VDD) -> VBUS
- D17 pad 3: Net-(D10-VDD) -> VBUS
- D18 pad 3: Net-(D10-VDD) -> VBUS
- D19 pad 3: Net-(D10-VDD) -> VBUS
- D20 pad 3: Net-(D10-VDD) -> VBUS
- D3 pad 3: Net-(D10-VDD) -> VBUS
- D4 pad 3: Net-(D10-VDD) -> VBUS
- D5 pad 3: Net-(D10-VDD) -> VBUS
- D6 pad 3: Net-(D10-VDD) -> VBUS
- D7 pad 3: Net-(D10-VDD) -> VBUS
- D8 pad 3: Net-(D10-VDD) -> VBUS
- D9 pad 3: Net-(D10-VDD) -> VBUS
- JP3 pad 2: Net-(D10-VDD) -> VBUS
- U8 pad 1: Net-(J6-Pin_2) -> /RSR_SCL
- U8 pad 2: Net-(J6-Pin_1) -> /RSR_3V
- U8 pad 3: Net-(J6-Pin_4) -> /RSR_GND
- U8 pad 4: Net-(J6-Pin_3) -> /RSR_SDA
Other:
- board outline added: 250 x 25 mm

Commit message: Add final footprint positions
Parts:
- added C28: 100nF, Capacitor_SMD:C_0603_1608Metric, B.Cu at (254.7, 60.0)
- added REF**: 15mm_played_slot, besser_footprints:15mm_played_slot, F.Cu at (248.5, 54.0)
- added REF**: 8mm_slot, besser_footprints:8mm_slot, F.Cu at (240.0, 58.4)
- added REF**: 8mm_slot, besser_footprints:8mm_slot, F.Cu at (257.0, 58.4)
- C1, C2, C3, C4, C5, C6, C8, C9, D1, D2, J2, J3, J4, J6, JP1, JP2, R1, R2, R3, R4, R5, SW1, SW2, U2, U3, U4, U5, U7: moved to B.Cu
- moved D20 245.7 mm to (253.2, 80.1)
- moved R3 241.5 mm to (273.4, 45.1), turned to 180 degrees
- moved D19 236.8 mm to (241.2, 80.1)
- moved R4 236.5 mm to (273.4, 57.9), turned to 180 degrees
- moved JP3 228.7 mm to (263.2, 80.1)
- moved D18 228.4 mm to (229.2, 80.1)
- moved C27 221.6 mm to (258.2, 81.1), turned to -90 degrees
- moved D2 221.4 mm to (267.5, 49.1)
- moved U8 220.8 mm to (249.1, 61.5)
- moved D17 220.5 mm to (217.2, 80.1)
- moved J6 216.1 mm to (250.5, 59.0), turned to 90 degrees
- moved C26 209.1 mm to (245.4, 81.1), turned to -90 degrees
- moved C25 198.1 mm to (233.9, 80.6), turned to -90 degrees
- moved J5 197.2 mm to (232.4, 58.4), turned to 90 degrees
- moved D16 190.0 mm to (204.7, 80.5)
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Connections:
- R5 pad 2: 3V3 -> 3V3_MCU
- U1 pad 15: /SDA -> /SCL
- U1 pad 16: unconnected-(U1-IO46-Pad16) -> /SDA
- U1 pad 17: unconnected-(U1-IO9-Pad17) -> /NEO_MCU
- U1 pad 38: /SCL -> unconnected-(U1-IO2-Pad38)
- U1 pad 6: /NEO_MCU -> unconnected-(U1-IO6-Pad6)
Routing:
- net (no net): vias 0 -> 4
- added copper zone on In1.Cu, net GND
- added copper zone on In2.Cu, net GND
Other:
- copper layers 2 -> 4
- rule pad_to_mask_clearance: 0 -> 0.04
- board text added: "10"
- board text added: "11"
- board text added: "12"
- board text added: "13"
- board text added: "14"
- board text added: "2¹"
- board text added: "3V3"
- board text added: "Board Flipped"
- board text added: "GND"
- board text added: "USB"
- board text added: "remap schematic so pins are more accessible"
- board text removed: "2²"

Commit message: Change schematic, start routing
Parts:
- removed JP1, JP2: SolderJumper_2_Bridged, besser_footprints:solder_jumper_bridged
- moved R1 36.3 mm to (90.0, 60.2), turned to 90 degrees
- moved R2 33.3 mm to (88.1, 60.2), turned to 90 degrees
- moved D2 4.80 mm to (267.7, 53.9)
- moved J2 1.60 mm to (122.1, 44.5)
- moved U4 1.60 mm to (125.4, 53.1)
- moved R5 1.06 mm to (70.8, 42.6), turned to 90 degrees
- moved D1 0.21 mm to (63.5, 50.9)
- moved C7 0.14 mm to (149.4, 61.9)
- moved C6 0.11 mm to (109.0, 58.6)
- moved U5 0.10 mm to (106.6, 51.5)
- turned C2 to 90 degrees
Connections:
- C1 pad 1: 3V3 -> 3V3_MCU
- U1 pad 15: /SCL -> /PPS
- U1 pad 16: /SDA -> unconnected-(U1-IO46-Pad16)
- U1 pad 31: unconnected-(U1-IO38-Pad31) -> /NEO_DISP
- U1 pad 32: unconnected-(U1-MTCK/IO39-Pad32) -> /SDA
- U1 pad 33: unconnected-(U1-MTDO/IO40-Pad33) -> /SCL
- U1 pad 36: /M_RX -> unconnected-(U1-RXD0/IO44-Pad36)
- U1 pad 37: /M_TX -> unconnected-(U1-TXD0/IO43-Pad37)
- U1 pad 4: /NEO_DISP -> unconnected-(U1-IO4-Pad4)
- U1 pad 5: /PPS -> unconnected-(U1-IO5-Pad5)
- U1 pad 7: /3V_EN -> unconnected-(U1-IO7-Pad7)
- U3 pad 3: /3V_EN -> VBUS
- U4 pad 2: Net-(JP2-B) -> unconnected-(U4-TXD-Pad2)
- U4 pad 3: Net-(JP1-B) -> unconnected-(U4-RXD-Pad3)
Routing:
- net /D-: track 0.00 -> 229.6 mm
- net /D+: track 0.00 -> 228.2 mm
- net /SCL: track 0.00 -> 209.2 mm, vias 0 -> 1
- net /SDA: track 0.00 -> 207.2 mm, vias 0 -> 1
- net VBUS: track 0.00 -> 204.9 mm
- net 3V3: track 0.00 -> 169.5 mm, vias 0 -> 1
- net /PPS: track 0.00 -> 79.7 mm, vias 0 -> 4
- net 3V3_MCU: track 0.00 -> 64.5 mm, vias 0 -> 4
- net GND: track 0.00 -> 59.5 mm, vias 0 -> 50
- net /NEO_DISP: track 0.00 -> 44.9 mm
- net /RESET: track 0.00 -> 39.1 mm, vias 0 -> 2
- net /BOOT: track 0.00 -> 32.9 mm
- net Net-(D2-A): track 0.00 -> 13.6 mm, vias 0 -> 4
- net /RSR_SCL: track 0.00 -> 8.62 mm, vias 0 -> 1
- net /NEO_MCU: track 0.00 -> 8.07 mm
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Other:
- rule solder_mask_min_width: 0.1 -> 0.12
- board text added: "Delete second LDO and swap RTC and GPS positions"

Commit message: Almost finish placements
Parts:
- C2, C3, C4, C5: value 10uF -> 1uF
- NEO VBUS: renamed from JP3
- moved D3 39.2 mm to (33.9, 44.4)
- moved D20 38.9 mm to (268.2, 44.2)
- moved D4 37.9 mm to (47.7, 45.1)
- moved D19 37.8 mm to (254.4, 44.7)
- moved C10 37.4 mm to (35.6, 48.0), turned to 0 degrees
- moved D18 37.2 mm to (240.6, 44.7)
- moved D5 37.0 mm to (61.5, 45.1)
- moved C11 36.9 mm to (49.4, 48.7), turned to 0 degrees
- moved D17 36.7 mm to (226.9, 44.7)
- moved D16 36.4 mm to (213.1, 45.1)
- moved D6 36.3 mm to (75.2, 45.1)
- moved D15 36.1 mm to (199.3, 45.1)
- moved D7 36.0 mm to (89.0, 45.0)
- moved D14 36.0 mm to (185.5, 45.1)
- moved D13 35.7 mm to (171.7, 45.1)
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Connections:
- J3 pad 2: VBUS -> 3V3
- J3 pad 3: 3V3 -> VBUS
- U1 pad 15: /PPS -> unconnected-(U1-IO3-Pad15)
- U1 pad 34: unconnected-(U1-MTDI/IO41-Pad34) -> /PPS
Routing:
- net 3V3: track 169.5 -> 208.2 mm, vias 1 -> 5
- net VBUS: track 204.9 -> 230.1 mm
- net /IO10: track 0.00 -> 18.8 mm
- net /PPS: track 79.7 -> 63.7 mm, vias 4 -> 2
- net /IO11: track 0.71 -> 16.4 mm
- net /IO12: track 0.36 -> 12.6 mm
- net /SCL: track 209.2 -> 199.2 mm, vias 1 -> 2
- net /IO13: track 0.11 -> 9.95 mm
- net /SDA: track 207.2 -> 198.4 mm, vias 1 -> 2
- net /IO14: track 0.40 -> 7.51 mm
- net /D-: track 229.6 -> 231.4 mm
- net /D+: track 228.2 -> 230.0 mm
- net /NEO_MCU: track 8.07 -> 8.93 mm
Other:
- board text added: "2²"
- board text added: "2³"
- board text added: "2⁰"
- board text added: "2⁴"
- board text added: "2⁵"
- board text added: "C10-C27"
- board text added: "D3-D20"
- board text added: "Hours"
- board text added: "Minutes"
- board text added: "Seconds"
- board text added: "https://youtu.be/PlXd3lLZ4vc?si=FWp1M6_FGoRUhZ_F&t=8296 2:18:16 have power and ground layers on top and bottom"
