File: binary_clock_PCB/binary_clock.kicad_sch (KiCad schematic)
At the start: 20 parts, among them J1 USB_C_Receptacle_USB2.0_16P, U1 ESP32-S3R8, U2 AP2112K-3.3, U3 MAX-M10S, U4 ESP32-WROOM-32E-R2, U5 SN74LVC1T45GW, U6 W25Q128JVPIQ

Commit message: Update
Parts:
- removed C9: 100nF, symbol Device:C
- removed U1: ESP32-S3R8, Package_DFN_QFN:QFN-56-1EP_7x7mm_P0.4mm_EP4x4mm, symbol MCU_Espressif:ESP32-S3
- removed U4: ESP32-WROOM-32E-R2, RF_Module:ESP32-WROOM-32D, symbol RF_Module:ESP32-WROOM-32E-R2
- removed U6: W25Q128JVPIQ, WSON_128JVPIQ_WIN, symbol W25Q128JVPIQ:W25Q128JVPIQ
- added R3, R4: 10K, symbol Device:R
- added R5: 5.1K, symbol Device:R
- added SW1, SW2: SW_DPST_x2, symbol Switch:SW_DPST_x2
- added U1: ESP32-S3-WROOM-2-N32R8V, RF_Module:ESP32-S3-WROOM-2, symbol RF_Module:ESP32-S3-WROOM-2
- added U6: DS3231M, Package_SO:SOIC-16W_7.5x10.3mm_P1.27mm, symbol Timer_RTC:DS3231M
- C2, C8: value 100nF -> 10uF
- U5: footprint Package_TO_SOT_SMD:SOT-563 -> Package_TO_SOT_SMD:SOT-363_SC-70-6
Connections:
- net 3V3: now also C6.2, U5.1 (VCCA), R3.1, R4.1, R5.2, U1.2 (3V3); no longer C6.1, C7.1
- net D+: now also U1.14 (USB_D+/IO20)
- net D-: now also U1.13 (USB_D-/IO19)
- net GND: now also U5.2 (GND), SW1.1 (A), SW2.2 (B), U1.1 (GND), U1.40 (GND), U1.41 (GND), U6.10 (GND), U6.11 (GND), U6.12 (GND), U6.13 (GND), U6.14 (VBAT), U6.5 (GND), U6.6 (GND), U6.7 (GND), U6.8 (GND), U6.9 (GND); no longer C6.2
- net VBUS: now also U5.5 (DIR), U5.6 (VCCB)
- net NEO: now reaches U5.3 (A)
- net NEO: now also U1.4 (IO4)
- net NEO_5V: now reaches U5.4 (B)
- new net: R4.2, U6.15 (SDA)
- new net: C6.1, U6.2 (VCC)
- new net: R3.2, U6.16 (SCL)
- new net BOOT: SW1.2 (B), U1.27 (IO0)
- new net RESET: C7.1, R5.1, SW2.1 (A), U1.3 (EN)
- new net SCL: U1.38 (IO2)
- new net SDA: U1.15 (IO3)
Other:
- note added: "Clean up schematic part labels"
- note added: "Ensure part designators are reset. They only count up, and dont go down as parts are deleted."
- note added: "MCU"
- note removed: "Ensure Part designators are reset. They only count up, and dont go down as parts are deleted."
- note removed: "Footprint might be incorrect Also make the symbol not stupid huge"
- moved on the sheet: C1, C2, C5, U3, U5

Commit message: Update
Parts:
- removed R3, R4: 10K, symbol Device:R
- added C11, C7, C9: 1uF, symbol Device:C
- added D1: SK6812, LED_SMD:LED_SK6812_PLCC4_5.0x5.0mm_P3.2mm, symbol LED:SK6812
- added J2: uFL, symbol Connector:Conn_Coaxial
- added J3: Conn_01x04_Socket, symbol Connector:Conn_01x04_Socket
- added J4: Conn_01x06_Socket, symbol Connector:Conn_01x06_Socket
- added R1, R2: 5.1K, symbol Device:R
- added U5: AP2112K-3.3, Package_TO_SOT_SMD:SOT-23-5, symbol Regulator_Linear:AP2112K-3.3
- added U7: VEML7700-TT, VEML7700-TT:XDCR_VEML7700-TT, symbol VEML7700-TT:VEML7700-TT
- C1: renamed from C4; value 100nF -> 1uF
- C5: renamed from C3; value 100nF -> 1uF
- renumbered C7 to C10, C8 to C2, C2 to C3, C5 to C4, C1 to C6, C6 to C8, D1 to D2, D2 to D3, R2 to R3, R1 to R4, U5 to U2, U2 to U3, U3 to U4
Connections:
- net 3V3: now also U4.7 (VCC_IO), U4.8 (VCC), C11.1, C9.1, R1.2, R2.2, U5.5 (VOUT), U7.2 (VDD); no longer C5.1, U1.2 (3V3), U3.5 (VOUT)
- net GND: now also U4.1 (GND), U4.10 (GND), U4.12 (GND), C7.1, C9.2, D1.1 (VSS), J2.2 (Ext), J3.4 (Pin_4), U5.2 (GND), U7.3 (GND)
- net SCL: now also U4.17 (SCL), U6.16 (SCL), J3.2 (Pin_2), R1.1, U7.1 (SCL)
- net SDA: now also U4.16 (SDA), U6.15 (SDA), J3.3 (Pin_3), R2.1, U7.4 (SDA)
- net VBUS: now also C7.2, U5.1 (VIN)
- net at U4.11 (RF_IN): now also J2.1 (In)
- net PPS: now reaches U4.4 (TIMEPULSE)
- net PPS: now also U1.5 (IO5)
- net NEO_MCU: now reaches U1.17 (IO9)
- net NEO_MCU: now also D1.2 (DIN)
- net 3V_EN: now reaches U1.7 (IO7)
- net 3V_EN: now also U5.3 (EN)
- net SHLD: no longer names the net of J1.S1 (SHIELD)
- new net: C11.2, J3.1 (Pin_1)
- new net 3V3_MCU: C5.1, D1.3 (VDD), U1.2 (3V3), U3.5 (VOUT)
- no-connect marks 0 -> 5
Other:
- note added: "3V3"
- note added: "MCU 3V3"
- note added: "Status"
- note added: "Switches"
- note added: "Timekeeping and Light Sensor"
- note added: "Try to compile custom CircuitPython build so that things like blinking red neopixel on error works, and being able to toggle I2C LDO (on by default, but can be turned off in code). https://learn.adafruit.com/how-to-add-a-new-board-to-circuitpython/customizing-the-board-files"
- note added: "USB-C"
- moved on the sheet: C1, C10, C5, C6, C8, D2, D3, J1, R3, R4, R5, SW1A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

Commit message: Update gitignore, PCB
Parts:
- removed C2, C3: 10uF, symbol Device:C
- removed C6: 100nF, symbol Device:C
- removed J4: Conn_01x06_Socket, symbol Connector:Conn_01x06_Socket
- removed SW1, SW2: SW_DPST_x2, symbol Switch:SW_DPST_x2
- added C10, C11, C12, C13, C14, C15, C16, C17, C18, C19, C20, C21, C22, C23, C24, C25, C26, C27, C7: 100nF, Capacitor_SMD:C_0603_1608Metric, symbol Device:C
- added D10, D11, D12, D13, D14, D15, D16, D17, D18, D19, D20, D4, D5, D6, D7, D8, D9: SK6812, LED_SMD:LED_SK6812_PLCC4_5.0x5.0mm_P3.2mm, symbol LED:SK6812
- added J3: Conn_01x08_Socket, Connector_PinHeader_2.54mm:PinHeader_1x08_P2.54mm_Vertical, symbol Connector:Conn_01x08_Socket
- added J6: Conn_01x04_Socket, symbol Connector:Conn_01x04_Socket
- added JP1, JP2, JP3: SolderJumper_2_Bridged, besser_footprints:solder_jumper_bridged, symbol Jumper:SolderJumper_2_Bridged
- added SW1, SW2: SW_SPST, symbol Switch:SW_SPST
- added U8: VEML7700-TT, VEML7700-TT:XDCR_VEML7700-TT, symbol VEML7700-TT:VEML7700-TT
- C1: renamed from C4; footprint (none) -> Capacitor_SMD:C_0603_1608Metric
- C2: renamed from C1; value 1uF -> 10uF; footprint (none) -> Capacitor_SMD:C_0603_1608Metric
- C3: renamed from C5; value 1uF -> 10uF; footprint (none) -> Capacitor_SMD:C_0603_1608Metric
- C4: renamed from C7; value 1uF -> 10uF; footprint (none) -> Capacitor_SMD:C_0603_1608Metric
- C5: renamed from C9; value 1uF -> 10uF; footprint (none) -> Capacitor_SMD:C_0603_1608Metric
- C6: renamed from C8; footprint (none) -> Capacitor_SMD:C_0603_1608Metric
- C8: renamed from C10; footprint (none) -> Capacitor_SMD:C_0603_1608Metric
- C9: renamed from C11; footprint (none) -> Capacitor_SMD:C_0603_1608Metric
- R1, R2, R5: footprint (none) -> Capacitor_SMD:C_0603_1608Metric
- R3: renamed from R4; footprint (none) -> Capacitor_SMD:C_0603_1608Metric
- R4: renamed from R3; footprint (none) -> Capacitor_SMD:C_0603_1608Metric
- renumbered D3 to D2, D2 to D3, J3 to J4, U3 to U2, U5 to U3, U6 to U5, U7 to U6, U2 to U7
Connections:
- net NEO_5V is gone; now on net NEO_5VLL: U7.4 (B)
- net 3V3: now also C6.1, C9.2, J4.1 (Pin_1), U5.2 (VCC), C7.2, J3.3 (Pin_3); no longer C6.2, C9.1
- net BOOT: now also SW1.1 (A)
- net GND: now also C6.2, C9.1, D3.1 (VSS), C10.1, C11.1, C12.1, C13.1, C14.1, C15.1, C16.1, C17.1, C18.1, C19.1, C20.1, C21.1, C22.1, C23.1, C24.1, C25.1, C26.1, C27.1, C7.1, D10.1 (VSS), D11.1 (VSS), D12.1 (VSS), D13.1 (VSS), D14.1 (VSS), D15.1 (VSS), D16.1 (VSS), D17.1 (VSS), D18.1 (VSS), D19.1 (VSS), D20.1 (VSS), D4.1 (VSS), D5.1 (VSS), D6.1 (VSS), D7.1 (VSS), D8.1 (VSS), D9.1 (VSS), J3.1 (Pin_1), SW1.2 (B), SW2.1 (A)
- net NEO_MCU: now also U1.6 (IO6); no longer U1.17 (IO9)
- net RESET: now also SW2.2 (B)
- net VBUS: now also C10.2, C11.2, C12.2, C13.2, C14.2, C15.2, C16.2, C17.2, C18.2, C19.2, C20.2, C21.2, C22.2, C23.2, C24.2, C25.2, C26.2, C27.2, J3.2 (Pin_2), JP3.1 (A)
- net at U4.2 (TXD): now also JP2.2 (B)
- net at U4.3 (RXD): now also JP1.2 (B)
- net IO10: now reaches U1.18 (IO10)
- net IO10: now also J3.4 (Pin_4)
- net IO11: now reaches U1.19 (IO11)
- net IO11: now also J3.5 (Pin_5)
- net IO12: now reaches U1.20 (IO12)
- net IO12: now also J3.6 (Pin_6)
- net IO13: now reaches U1.21 (IO13)
- net IO13: now also J3.7 (Pin_7)
- net IO14: now reaches U1.22 (IO14)
- net IO14: now also J3.8 (Pin_8)
- net M_RX: now reaches U1.36 (RXD0/IO44)
- net M_RX: now also JP2.1 (A)
- net M_TX: now reaches U1.37 (TXD0/IO43)
- net M_TX: now also JP1.1 (A)
- net NEO_5VLL: now reaches D3.2 (DIN)
- net at D3.3 (VDD): now also D10.3 (VDD), D11.3 (VDD), D12.3 (VDD), D13.3 (VDD), D14.3 (VDD), D15.3 (VDD), D16.3 (VDD), D17.3 (VDD), D18.3 (VDD), D19.3 (VDD), D20.3 (VDD), D4.3 (VDD), D5.3 (VDD), D6.3 (VDD), D7.3 (VDD), D8.3 (VDD), D9.3 (VDD), JP3.2 (B)
- net at D3.4 (DOUT): now also D4.2 (DIN)
- net CC1: no longer names the net of J1.A5 (CC1), R3.1
- net CC2: no longer names the net of J1.B5 (CC2), R4.1
- net NEO renamed NEO_DISP
- new net: D16.4 (DOUT), D17.2 (DIN)
- new net: D17.4 (DOUT), D18.2 (DIN)
- new net: D10.4 (DOUT), D11.2 (DIN)
- new net: D11.4 (DOUT), D12.2 (DIN)
- new net: D19.4 (DOUT), D20.2 (DIN)
- new net: D6.4 (DOUT), D7.2 (DIN)
- new net: D7.4 (DOUT), D8.2 (DIN)
- new net: D4.4 (DOUT), D5.2 (DIN)
- new net: D5.4 (DOUT), D6.2 (DIN)
- new net: D8.4 (DOUT), D9.2 (DIN)
- new net: D10.2 (DIN), D9.4 (DOUT)
- new net: J6.2 (Pin_2), U8.1 (SCL)
- new net: J6.1 (Pin_1), U8.2 (VDD)
- new net: J6.4 (Pin_4), U8.3 (GND)
- new net: J6.3 (Pin_3), U8.4 (SDA)
- new net: D13.4 (DOUT), D14.2 (DIN)
- new net: D14.4 (DOUT), D15.2 (DIN)
- new net: D15.4 (DOUT), D16.2 (DIN)
- new net: D12.4 (DOUT), D13.2 (DIN)
- new net: D18.4 (DOUT), D19.2 (DIN)
- no-connect marks 5 -> 32
Other:
- note added: "50Ω impedance"
- note added: "GPIO"
- note added: "In case the normal position of the light sensor is sheilded by the case, this can be popped off the PCB and have the light sensor and Qwicc connector attached. Do not place the light sensor or Qwiic connector."
- note added: "Neopixel Display"
- note added: "Qwiic"
- note added: "Riser"
- note added: "Use 0602 pad with exposed trace for jumper"
- company: (none) -> besser
- moved on the sheet: C1, C6, C8, C9, D2, D3, J2, J4, R1, R2, R3, R5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

Commit message: Update PCB
Parts:
- added J5: JST-SM04B-SRSS, besser_footprints:JST_SH_SM04B-SRSS-TB_1x04-1MP_P1.00mm_Horizontal, symbol Connector:Conn_01x04_Socket
- J1: value USB_C_Receptacle_USB2.0_16P -> USB4105-GF-A; footprint (none) -> Connector_USB:USB_C_Receptacle_GCT_USB4105-xx-A_16P_TopMnt_Horizontal
- J2: footprint (none) -> Connector_Coaxial:U.FL_Hirose_U.FL-R-SMT-1_Vertical
- J4, J6: value Conn_01x04_Socket -> JST-SM04B-SRSS; footprint (none) -> besser_footprints:JST_SH_SM04B-SRSS-TB_1x04-1MP_P1.00mm_Horizontal
- U6: footprint VEML7700-TT:XDCR_VEML7700-TT -> besser_footprints:VEML7700
- U8: now in the parts list
Connections:
- net 3V3: now also C9.1, J4.2 (Pin_2), J5.2 (Pin_2); no longer C9.2, J4.1 (Pin_1)
- net GND: now also C9.2, J4.1 (Pin_1), J5.1 (Pin_1); no longer C9.1, J4.4 (Pin_4)
- net SCL: now also J4.4 (Pin_4), J5.4 (Pin_4); no longer J4.2 (Pin_2)
- net SDA: now also J5.3 (Pin_3)
- net RSR_3V: now reaches J6.2 (Pin_2)
- net RSR_3V: now also U8.2 (VDD); no longer U8.1 (SCL)
- net RSR_GND: now reaches J6.1 (Pin_1)
- net RSR_GND: now also U8.3 (GND); no longer U8.2 (VDD)
- net RSR_SCL: now reaches J6.4 (Pin_4)
- net RSR_SCL: now also U8.1 (SCL); no longer U8.3 (GND)
- net RSR_SDA: now reaches J6.3 (Pin_3), U8.4 (SDA)
Other:
- note added: "In case the normal position of the light sensor is sheilded by the case, this part of the PCB can be removed so the light sensor can be on a daughterboard for better light visibility. It is attached with a Qwiic connecter (JST-SH with I2C). This is to save cost from it being a seperate PCB."
- note added: "Light Sensor Riser"
- note removed: "In case the normal position of the light sensor is sheilded by the case, this can be popped off the PCB and have the light sensor and Qwicc connector attached. Do not place the light sensor or Qwiic connector."
- note removed: "Riser"
- note removed: "Use 0602 pad with exposed trace for jumper"
- moved on the sheet: J4, U8

Commit message: Start on PCB
Parts:
- SW1, SW2: value SW_SPST -> PTS636 SK25F; footprint (none) -> Button_Switch_SMD:SW_Tactile_SPST_NO_Straight_CK_PTS636Sx25SMTRLFS
- U8: footprint VEML7700-TT:XDCR_VEML7700-TT -> besser_footprints:VEML7700
Connections:
- net VBUS: now also D10.3 (VDD), D11.3 (VDD), D12.3 (VDD), D13.3 (VDD), D14.3 (VDD), D15.3 (VDD), D16.3 (VDD), D17.3 (VDD), D18.3 (VDD), D19.3 (VDD), D20.3 (VDD), D3.3 (VDD), D4.3 (VDD), D5.3 (VDD), D6.3 (VDD), D7.3 (VDD), D8.3 (VDD), D9.3 (VDD), JP3.2 (B)
- net ANT: now reaches J2.1 (In), U4.11 (RF_IN)
- net CC1: now reaches J1.A5 (CC1), R3.1
- net CC2: now reaches J1.B5 (CC2), R4.1
Other:
- note removed: "Clean up schematic part labels"
- note removed: "Ensure part designators are reset. They only count up, and dont go down as parts are deleted."
Changed lines of the file:
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@@
 	(wire
 		(pts
+			(xy 53.34 196.85) (xy 63.5 196.85)
+		)
+		(stroke
+			(width 0)
+			(type default)
+		)
+	)
+	(wire
+		(pts
 			(xy 261.62 27.94) (xy 280.67 27.94)
 		)
@@
 	(wire
 		(pts
-			(xy 53.34 196.85) (xy 63.5 196.85)
-		)
-		(stroke
-			(width 0)
-			(type default)
-		)
-	)
-	(wire
-		(pts
 			(xy 309.88 241.3) (xy 303.53 241.3)
 		)
@@
 	(wire
 		(pts
-			(xy 153.67 241.3) (xy 153.67 238.76)
+			(xy 148.59 181.61) (xy 162.56 181.61)
 		)
 		(stroke
@@
 		)
 	)
-	(polyline
+	(wire
 		(pts
-			(xy 299.72 189.23) (xy 299.72 224.79)
+			(xy 153.67 241.3) (xy 153.67 238.76)
 		)
 		(stroke
 			(width 0)
-			(type dash)
+			(type default)
 		)
 	)
-	(wire
+	(polyline
 		(pts
-			(xy 148.59 181.61) (xy 162.56 181.61)
+			(xy 299.72 189.23) (xy 299.72 224.79)
 		)
 		(stroke
 			(width 0)
-			(type default)
+			(type dash)
 		)
 	)
@@
 	(text "50Ω impedance"
 		(exclude_from_sim no)
-		(at 176.784 256.794 0)
+		(at 176.022 261.112 0)
 		(effects
 			(font
-				(size 1.524 1.524)
+				(size 1.143 1.143)
 			)
 		)
@@
 		)
 	)
-	(text "Clean up schematic part labels"
-		(exclude_from_sim no)
-		(at 241.808 121.666 0)
-		(effects
-			(font
-				(size 5.08 5.08)
-			)
-		)
-	)
 	(text "Status"
 		(exclude_from_sim no)
@@
 		)
 	)
-	(text "Ensure part designators are reset.\nThey only count up, and dont go down as parts are deleted."
-		(exclude_from_sim no)
-		(at 194.31 102.108 0)
-		(effects
-			(font
-				(size 5.08 5.08)
-			)
-			(justify left)
-		)
-	)
 	(text "Qwiic\n"
 		(exclude_from_sim no)
@@
 	(text "Try to compile custom CircuitPython build so that things\nlike blinking red neopixel on error works, and being able to\ntoggle I2C LDO (on by default, but can be turned off in code).\n\nhttps://learn.adafruit.com/how-to-add-a-new-board-to-circuitpython/customizing-the-board-files"
 		(exclude_from_sim no)
-		(at 12.7 165.608 0)
+		(at 85.09 117.348 0)
 		(effects
 			(font
@@
 		)
 	)
+	(label "VBUS"
+		(at 46.99 27.94 0)
+		(fields_autoplaced yes)
+		(effects
+			(font
+				(size 1.27 1.27)
+			)
+			(justify left bottom)
+		)
+	)
 	(label "D-"
 		(at 63.5 240.03 180)
@@
 		)
 	)
+	(label "SCL"
+		(at 63.5 196.85 180)
+		(fields_autoplaced yes)
+		(effects
+			(font
+				(size 1.27 1.27)
+			)
+			(justify right bottom)
+		)
+	)
 	(label "IO12"
 		(at 264.16 175.26 0)
@@
 		)
 	)
+	(label "CC2"
+		(at 149.86 184.15 0)
+		(fields_autoplaced yes)
+		(effects
+			(font
+				(size 1.27 1.27)
+			)
+			(justify left bottom)
+		)
+	)
 	(label "SCL"
 		(at 303.53 241.3 0)
@@
 		)
 	)
+	(label "CC1"
+		(at 149.86 181.61 0)
+		(fields_autoplaced yes)
+		(effects
+			(font
+				(size 1.27 1.27)
+			)
+			(justify left bottom)
+		)
+	)
 	(label "SCL"
 		(at 91.44 186.69 0)
@@
 		)
 	)
+	(label "ANT"
+		(at 175.26 259.08 0)
+		(fields_autoplaced yes)
+		(effects
+			(font
+				(size 1.27 1.27)
+			)
+			(justify left bottom)
+		)
+	)
 	(label "M_TX"
 		(at 63.5 260.35 180)
@@
 		)
 	)
-	(label "SCL"
-		(at 63.5 196.85 180)
-		(fields_autoplaced yes)
-		(effects
-			(font
-				(size 1.27 1.27)
-			)
-			(justify right bottom)
-		)
-	)
 	(label "IO10"
 		(at 63.5 217.17 180)
@@
 			)
 		)
-		(property "Footprint" "VEML7700-TT:XDCR_VEML7700-TT"
+		(property "Footprint" "besser_footprints:VEML7700"
 			(at 361.95 213.36 0)
 			(effects
@@
 			)
 		)
-		(property "Value" "SW_SPST"
+		(property "Value" "PTS636 SK25F"
 			(at 196.85 205.74 0)
 			(effects
@@
 			)
 		)
-		(property "Footprint" ""
+		(property "Footprint" "Button_Switch_SMD:SW_Tactile_SPST_NO_Straight_CK_PTS636Sx25SMTRLFS"
 			(at 196.85 209.55 0)
 			(effects
@@
 			)
 		)
-		(property "Value" "SW_SPST"
+		(property "Value" "PTS636 SK25F"
 			(at 227.33 205.74 0)
 			(effects
@@
 			)
 		)
-		(property "Footprint" ""
+		(property "Footprint" "Button_Switch_SMD:SW_Tactile_SPST_NO_Straight_CK_PTS636Sx25SMTRLFS"
 			(at 227.33 209.55 0)
 			(effects
