File: binary_clock_PCB/binary_clock.kicad_sch (KiCad schematic)
At the start: 70 parts, among them J1 USB4105-GF-A, J2 uFL, J3 Conn_01x08_Socket, J4 JST-SM04B-SRSS, J5 JST-SM04B-SRSS, J6 JST-SM04B-SRSS, SW1 PTS636 SK25F, SW2 PTS636 SK25F, U1 ESP32-S3-WROOM-2-N32R8V, U2 AP2112K-3.3, U3 AP2112K-3.3, U4 MAX-M10S, U5 DS3231M, U6 VEML7700-TT, U7 SN74LVC1T45GW, U8 VEML7700-TT

Commit message: dead :pensive:
Connections:
- net 3V3: no longer U7.1 (VCCA)
- net 3V3_MCU: now also U7.1 (VCCA)
- net NEO_DISP: now also U1.15 (IO3); no longer U1.31 (IO38)
- net VBUS: no longer C10.2, C11.2, C12.2, C13.2, C14.2, C15.2, C16.2, C17.2, C18.2, C19.2, C20.2, C21.2, C22.2, C23.2, C24.2, C25.2, C26.2, C27.2, D10.3 (VDD), D11.3 (VDD), D12.3 (VDD), D13.3 (VDD), D14.3 (VDD), D15.3 (VDD), D16.3 (VDD), D17.3 (VDD), D18.3 (VDD), D19.3 (VDD), D20.3 (VDD), D3.3 (VDD), D4.3 (VDD), D5.3 (VDD), D6.3 (VDD), D7.3 (VDD), D8.3 (VDD), D9.3 (VDD), JP3.2 (B), U3.3 (EN), U7.5 (DIR), U7.6 (VCCB)
- new net 3V3_EN: U1.31 (IO38), U3.3 (EN)
- new net NEO_VBUS: C10.2, C11.2, C12.2, C13.2, C14.2, C15.2, C16.2, C17.2, C18.2, C19.2, C20.2, C21.2, C22.2, C23.2, C24.2, C25.2, C26.2, C27.2, D10.3 (VDD), D11.3 (VDD), D12.3 (VDD), D13.3 (VDD), D14.3 (VDD), D15.3 (VDD), D16.3 (VDD), D17.3 (VDD), D18.3 (VDD), D19.3 (VDD), D20.3 (VDD), D3.3 (VDD), D4.3 (VDD), D5.3 (VDD), D6.3 (VDD), D7.3 (VDD), D8.3 (VDD), D9.3 (VDD), JP3.2 (B), U7.5 (DIR), U7.6 (VCCB)
- no-connect marks 37 -> 36

Commit message: Add gerber files
Connections:
- net ALM: now reaches U5.3 (~{INT}/SQW)
- net ALM: now also U1.23 (IO21)
- no-connect marks 36 -> 34
Changed lines of the file:
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@@
-	)
-	(no_connect
-		(at 237.49 264.16)
 	)
 	(no_connect
@@
 	)
 	(no_connect
-		(at 53.34 245.11)
-	)
-	(no_connect
 		(at 53.34 232.41)
 	)
@@
 		)
 	)
+	(wire
+		(pts
+			(xy 237.49 264.16) (xy 245.11 264.16)
+		)
+		(stroke
+			(width 0)
+			(type default)
+		)
+	)
 	(polyline
 		(pts
@@
 		(pts
 			(xy 223.52 43.18) (xy 242.57 43.18)
+		)
+		(stroke
+			(width 0)
+			(type default)
+		)
+	)
+	(wire
+		(pts
+			(xy 53.34 245.11) (xy 63.5 245.11)
 		)
 		(stroke
@@
 		)
 	)
+	(label "ALM"
+		(at 63.5 245.11 180)
+		(fields_autoplaced yes)
+		(effects
+			(font
+				(size 1.27 1.27)
+			)
+			(justify right bottom)
+		)
+	)
 	(label "PPS"
 		(at 176.53 266.7 180)
@@
 		)
 	)
+	(label "ALM"
+		(at 245.11 264.16 180)
+		(fields_autoplaced yes)
+		(effects
+			(font
+				(size 1.27 1.27)
+			)
+			(justify right bottom)
+		)
+	)
