File: lightbeam_s3_PCB/lightbeam_s3.kicad_pcb (KiCad board)
At the start: 4 copper layers, 250 x 25 mm, 73 parts, among them J1 USB4105-GF-A, J2 uFL, J3 Conn_01x08_Socket, J4 JST-SM04B-SRSS, J5 JST-SM04B-SRSS, J6 JST-SM04B-SRSS, SW2 PTS636 SK25F, U1 ESP32-S3-WROOM-2-N32R8V, U2 AP2112K-3.3, U3 AP2112K-3.3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

Commit message: Increase diode to 2A
Other:
- board text added: "VBS"
- board text removed: "5V5"

Commit message: Fix I2C lines, remove edge power line
Parts:
- D2: value NSR0320MW2T1G -> PMEG1020EA
- moved C7 1.40 mm to (151.7, 61.9), turned to 0 degrees
- renumbered Boot to SW1
Connections:
- U1 pad 32: /SDA -> unconnected-(U1-MTCK/IO39-Pad32)
- U1 pad 33: /SCL -> unconnected-(U1-MTDO/IO40-Pad33)
- U1 pad 38: unconnected-(U1-IO2-Pad38) -> /SDA
- U1 pad 39: unconnected-(U1-IO1-Pad39) -> /SCL
Routing:
- net /SCL: track 195.5 -> 203.6 mm
- net /SDA: track 193.9 -> 202.0 mm
- net Net-(D2-A): track 13.6 -> 7.95 mm
- net /PPS: track 59.8 -> 56.4 mm
- net VBUS: track 240.5 -> 238.2 mm
- net 3V3: track 199.9 -> 197.7 mm
- net GND: track 106.3 -> 105.2 mm, vias 282 -> 294
- added copper zone on F.Cu, net Net-(D2-A)

Commit message: Improve grounding, move USB lines inward
Parts:
- moved C8 0.40 mm to (70.8, 47.8)
- moved R5 0.40 mm to (70.8, 43.0)
- moved SW2 0.40 mm to (75.0, 45.4)
Routing:
- net /D+: track 230.1 -> 228.3 mm
- net /D-: track 231.4 -> 230.4 mm
- net VBUS: track 238.2 -> 237.3 mm
- net 3V3_MCU: track 68.3 -> 67.5 mm
- net GND: vias 294 -> 299

Commit message: Improve PCB for the enclosure, clean traces, DNP GNSS
Parts:
- moved C7 0.70 mm to (151.7, 61.2)
- moved U6 0.70 mm to (153.6, 59.9)
Routing:
- net 3V3: track 197.7 -> 195.8 mm
- net /SCL: track 203.6 -> 204.4 mm
Other:
- board text added: "Light Sensor Riser"
